File: Projects/Williamson88/Williamson88.brd (EAGLE design)
At the start: 160 x 100 mm, 1 part

Commit message: Created schematic and first placement
Parts:
- added C1, C2, C3, C4: .22uF, rcl:C150-091X182
- added R1: (no value), pot:B25P
- added R10, R3, R9: 47k, rcl:0309/10
- added R11, R12: 100k, rcl:0309/10
- added R13, R14, R2: 10k, rcl:0309/10
- added R15, R16: 1k, rcl:0309/10
- added R17, R18: 10, rcl:0309/10
- added R19, R20: 10k, pot:B25P
- added R21: 680, rcl:0309/10
- added R4: 470, rcl:0309/10
- added R5: 22k, rcl:0309/10
- added R6: (no value), rcl:0309/10
- added R7, R8: 470k, rcl:0309/10
- added V2, V3, V4: (no value), tubes:OKTAL
- moved V1 77.9 mm to (43.2, 49.5), turned to 225 degrees
Connections:
- new net -80V: R19.E, R20.E
- new net 230V: R3.1
- new net 320V: R5.1
- new net 477V: R10.1, R9.2
- new net GND: R1.A, R13.2, R14.2, R17.1, R18.2, R21.1, R4.2, R6.2, R7.2, R8.1
- new net N$1: R3.2, V1.2, V1.4
- new net N$10: C3.1, R10.2, V2.5
- new net N$11: C4.1, R9.1, V2.2
- new net N$12: C3.2, R11.1, R15.1
- new net N$13: R15.2, V3.4
- new net N$14: C4.2, R12.2, R16.1
- new net N$15: R16.2, V4.4
- new net N$16: R17.2, V3.1
- new net N$17: R18.1, V4.1
- new net N$18: R13.1, R19.A
- new net N$19: R2.1, V1.1
- new net N$2: R4.1, V1.3
- new net N$20: R14.1, R20.A
- new net N$21: R12.1, R20.S
- new net N$22: R11.2, R19.S
- new net N$3: C2.1, R6.1, V1.6
- new net N$4: C1.1, R5.2, V1.5
- new net N$6: C1.2, R7.1, V2.4
- new net N$7: C2.2, R8.2, V2.1
- new net N$8: R1.S, R2.2
- new net N$9: R21.2, V2.3, V2.6
- new net T1A: V3.6
- new net T2A: V3.5
- new net T3A: V4.5
- new net T4A: V4.6
- new net VIN: R1.E
Other:
- board size 160 x 100 mm -> 207 x 100 mm

Commit message: Added attributes and MPN Created the power circuit
Parts:
- added CY1, CY2, CY4: 47u, rcl:E7,5-18
- added CY3: (no value), rcl:YC10B5
- added CY5, CY6: 1000u, rcl:E7,5-18
- added R22: 10k, rcl:0309/10
- C1, C2, C3, C4: device rcl:C150-091X182 -> rcl:C225-062X268
- R6: value (none) -> 22k
- V1, V2: value (none) -> 6SN7
- V3, V4: value (none) -> KT88
- moved R6 14.8 mm to (69.8, 53.3), turned to 0 degrees
- moved C2 6.35 mm to (69.8, 61.0)
- moved C1 5.24 mm to (71.1, 39.4)
- moved R7 5.24 mm to (81.3, 45.7), turned to 0 degrees
- moved C4 4.02 mm to (104.1, 55.9)
- moved R5 2.54 mm to (64.8, 33.0), turned to 180 degrees
Connections:
- new net FB: CY3.2, R22.2
- new net HEATERS_M: V1.8, V2.8, V3.2, V4.2
- new net HEATERS_P: V1.7, V2.7, V3.7, V4.7
- net 230V: now also CY1.+
- net 320V: now also CY2.+
- net 477V: now also CY4.-
- net GND: now also CY1.-, CY2.-, CY4.+, CY5.-, CY6.-
- net N$16: now also CY5.+
- net N$17: now also CY6.+
- net N$2: now also CY3.1, R22.1

Commit message: Created library for audio transformer
Parts:
- added U$1: CXPP30, CXPP30:CXPP30
- added U$10, U$11, U$12, U$13, U$14, U$15, U$2, U$3, U$4, U$5, U$6, U$7, U$8, U$9: W_CONN, CXPP30:WIRE_T
- moved R15 73.3 mm to (74.7, 66.2)
- moved V3 72.9 mm to (94.0, 73.7)
- moved R17 68.4 mm to (117.8, 67.5)
- moved R16 63.4 mm to (5.96, 67.5)
- moved V4 57.8 mm to (29.2, 73.7)
- moved R18 52.9 mm to (52.8, 73.7)
- moved V1 22.5 mm to (36.8, 27.9)
- moved R11 22.3 mm to (152.5, 23.1)
- moved R6 22.3 mm to (63.6, 32.0)
- moved C1 22.3 mm to (64.8, 18.0)
- moved C2 22.3 mm to (63.6, 39.6)
- moved C4 22.3 mm to (97.9, 34.5)
- moved R1 22.3 mm to (7.70, 39.6)
- moved R12 22.3 mm to (99.1, 25.6)
- moved R2 22.3 mm to (16.6, 37.1)
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Connections:
- removed net FB: CY3.2, R22.2
- new net 16O: CY3.2, R22.2, U$6.P$1
- new net 4O: U$8.P$1
- new net 8O: U$7.P$1
- new net COMMON: U$9.P$1
- net -80V: now also U$10.P$1
- net 230V: now also U$11.P$1
- net 320V: now also U$12.P$1
- net 477V: now also U$13.P$1
- net HEATERS_M: now also U$15.P$1
- net HEATERS_P: now also U$14.P$1
- net T1A: now also U$2.P$1
- net T2A: now also U$3.P$1
- net T3A: now also U$4.P$1
- net T4A: now also U$5.P$1
Other:
- board size 207 x 100 mm -> 180.3 x 211.8 mm

Commit message: Added library for audio caps
Parts:
- removed CY1, CY2, CY4: 47u, rcl:E7,5-18
- added U$16, U$17, U$18: W_CONN, CXPP30:WIRE_T
- moved U$14 228.5 mm to (137.7, 70.6), turned to 270 degrees
- moved U$15 227.1 mm to (137.7, 66.3), turned to 270 degrees
- moved U$5 193.2 mm to (16.5, 103.6), turned to 270 degrees
- moved U$4 191.0 mm to (19.8, 103.6), turned to 270 degrees
- moved U$3 188.9 mm to (23.4, 103.6), turned to 270 degrees
- moved U$2 186.9 mm to (26.9, 103.6), turned to 270 degrees
- moved U$1 176.0 mm to (203.5, 117.4)
- moved CY3 167.5 mm to (90.9, 119.9)
- moved CY5 161.3 mm to (120.7, 63.0), turned to 90 degrees
- moved R22 160.0 mm to (91.2, 124.7)
- moved R1 151.8 mm to (126.0, 134.7), turned to 270 degrees
- moved R3 146.2 mm to (123.5, 121.7), turned to 270 degrees
- moved R2 141.6 mm to (131.3, 120.1)
- moved R4 136.6 mm to (105.7, 122.4), turned to 0 degrees
- moved R10 107.6 mm to (72.8, 85.1), turned to 270 degrees
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Connections:
- new net 505V: U$18.P$1
- net 230V: no longer CY1.+
- net 320V: no longer CY2.+
- net 477V: now also U$16.P$1; no longer CY4.-
- net GND: no longer CY1.-, CY2.-, CY4.+
- net T2A: now also U$17.P$1
Other:
- board size 180.3 x 211.8 mm -> 140 x 210 mm

Commit message: Cleanup and schematic for the amplifier part
Parts:
- removed U$11, U$12, U$13, U$16: W_CONN, CXPP30:WIRE_T
- added CY1, CY2, CY4: 100uF, rcl:E7,5-18
- added R23: 22k, rcl:0309/10
- added R24: 27k, rcl:0309/10
- added R25: 4.7k, rcl:0309/10
- R22: value 10k -> 39k
- moved U$1 9.40 mm to (200.4, 126.3)
Connections:
- removed net 230V: R3.1, U$11.P$1
- removed net 505V: U$18.P$1
- new net 370V: CY1.+, R23.1, R24.2, R5.1
- new net 530V: R25.2, U$18.P$1
- net 320V: now also CY2.+, R24.1, R3.1; no longer R5.1, U$12.P$1
- net 477V: now also CY4.+, R23.2, R25.1; no longer U$13.P$1, U$16.P$1
- net GND: now also CY1.-, CY2.-, CY4.-
Changed lines of the file:
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@@
 <setting verticaltext="up"/>
 </settings>
-<grid distance="10" unitdist="mil" unit="mm" style="lines" multiple="1" display="yes" altdistance="10" altunitdist="mil" altunit="mm"/>
+<grid distance="10" unitdist="mil" unit="mil" style="lines" multiple="1" display="yes" altdistance="10" altunitdist="mil" altunit="mil"/>
 <layers>
 <layer number="1" name="Top" color="4" fill="1" visible="yes" active="yes"/>
@@
 <layer number="18" name="Vias" color="2" fill="1" visible="yes" active="yes"/>
 <layer number="19" name="Unrouted" color="6" fill="1" visible="yes" active="yes"/>
-<layer number="20" name="Dimension" color="15" fill="1" visible="yes" active="yes"/>
+<layer number="20" name="Dimension" color="24" fill="1" visible="yes" active="yes"/>
 <layer number="21" name="tPlace" color="7" fill="1" visible="yes" active="yes"/>
 <layer number="22" name="bPlace" color="7" fill="1" visible="yes" active="yes"/>
@@
 <wire x1="140" y1="210" x2="0" y2="210" width="0" layer="20"/>
 <wire x1="0" y1="210" x2="0" y2="0" width="0" layer="20"/>
-<circle x="27.686" y="27.94" radius="26" width="0.3048" layer="22"/>
+<circle x="26.67" y="27.94" radius="26" width="0.3048" layer="22"/>
 <circle x="110.998" y="101.854" radius="17" width="0.3048" layer="21"/>
 <circle x="110.998" y="27.94" radius="26" width="0.3048" layer="21"/>
@@
 <element name="R20" library="pot" package="B25P" value="10k" x="68.17" y="30.256" rot="R90"/>
 <element name="V2" library="tubes" package="OKTAL" value="6SN7" x="54.864" y="76.2" rot="R270"/>
-<element name="R22" library="rcl" package="0309/10" value="10k" x="91.186" y="124.714"/>
+<element name="R22" library="rcl" package="0309/10" value="39k" x="91.186" y="124.714"/>
 <element name="CY3" library="rcl" package="YC10B5" value="" x="90.932" y="119.888"/>
 <element name="CY5" library="rcl" package="E7,5-18" value="1000u" x="120.65" y="62.992" rot="R90">
@@
 <attribute name="RATING" value="50V" x="55.118" y="12.192" size="1.778" layer="27" rot="R270" display="off"/>
 </element>
-<element name="U$1" library="CXPP30" package="CXPP30" value="CXPP30" x="203.454" y="117.442"/>
+<element name="U$1" library="CXPP30" package="CXPP30" value="CXPP30" x="200.406" y="126.332"/>
 <element name="U$2" library="CXPP30" package="WIRE_T" value="W_CONN" x="26.924" y="103.632" rot="R270"/>
 <element name="U$3" library="CXPP30" package="WIRE_T" value="W_CONN" x="23.368" y="103.632" rot="R270"/>
@@
 <element name="U$9" library="CXPP30" package="WIRE_T" value="W_CONN" x="0" y="-99.06"/>
 <element name="U$10" library="CXPP30" package="WIRE_T" value="W_CONN" x="0" y="-101.6"/>
-<element name="U$11" library="CXPP30" package="WIRE_T" value="W_CONN" x="0" y="-104.14"/>
-<element name="U$12" library="CXPP30" package="WIRE_T" value="W_CONN" x="0" y="-106.68"/>
-<element name="U$13" library="CXPP30" package="WIRE_T" value="W_CONN" x="0" y="-109.22"/>
 <element name="U$14" library="CXPP30" package="WIRE_T" value="W_CONN" x="137.668" y="70.612" rot="R270"/>
 <element name="U$15" library="CXPP30" package="WIRE_T" value="W_CONN" x="137.668" y="66.294" rot="R270"/>
-<element name="U$16" library="CXPP30" package="WIRE_T" value="W_CONN" x="0" y="-116"/>
 <element name="U$17" library="CXPP30" package="WIRE_T" value="W_CONN" x="-0.254" y="-117.856"/>
 <element name="U$18" library="CXPP30" package="WIRE_T" value="W_CONN" x="-0.508" y="-119.634"/>
+<element name="R23" library="rcl" package="0309/10" value="22k" x="-58.674" y="-124.46"/>
+<element name="R24" library="rcl" package="0309/10" value="27k" x="-58.674" y="-129.794"/>
+<element name="R25" library="rcl" package="0309/10" value="4.7k" x="-58.674" y="-189.23">
+<attribute name="RATING" value="5W" x="-58.674" y="-189.23" size="1.778" layer="27" display="off"/>
+</element>
+<element name="CY2" library="rcl" package="E7,5-18" value="100uF" x="-55.372" y="-199.898">
+<attribute name="RATING" value="600V" x="-55.372" y="-199.898" size="1.778" layer="27" display="off"/>
+</element>
+<element name="CY1" library="rcl" package="E7,5-18" value="100uF" x="-55.372" y="-217.932">
+<attribute name="RATING" value="600V" x="-55.372" y="-217.932" size="1.778" layer="27" display="off"/>
+</element>
+<element name="CY4" library="rcl" package="E7,5-18" value="100uF" x="-55.372" y="-235.966">
+<attribute name="RATING" value="600V" x="-55.372" y="-235.966" size="1.778" layer="27" display="off"/>
+</element>
 </elements>
 <signals>
@@
 <contactref element="CY5" pad="-"/>
 <contactref element="CY6" pad="-"/>
+<contactref element="CY2" pad="-"/>
+<contactref element="CY1" pad="-"/>
+<contactref element="CY4" pad="-"/>
+<wire x1="-51.562" y1="-217.932" x2="-51.562" y2="-199.898" width="0" layer="19" extent="1-1"/>
+<wire x1="-51.562" y1="-235.966" x2="-51.562" y2="-217.932" width="0" layer="19" extent="1-1"/>
+<wire x1="43.392" y1="5.668" x2="-51.562" y2="-199.898" width="0" layer="19" extent="1-1"/>
+<wire x1="55.118" y1="8.382" x2="43.392" y2="5.668" width="0" layer="19" extent="1-1"/>
+<wire x1="78.298" y1="22.89" x2="55.118" y2="8.382" width="0" layer="19" extent="1-1"/>
+<wire x1="80.452" y1="38.07" x2="78.298" y2="22.89" width="0" layer="19" extent="1-1"/>
+<wire x1="95.062" y1="57.434" x2="80.452" y2="38.07" width="0" layer="19" extent="1-1"/>
+<wire x1="95.062" y1="62.768" x2="95.062" y2="57.434" width="0" layer="19" extent="1-1"/>
+<wire x1="99.03" y1="62.804" x2="95.062" y2="62.768" width="0" layer="19" extent="1-1"/>
+<wire x1="94.966" y1="78.298" x2="95.062" y2="62.768" width="0" layer="19" extent="1-1"/>
+<wire x1="108.11" y1="45.522" x2="95.062" y2="57.434" width="0" layer="19" extent="1-1"/>
+<wire x1="120.65" y1="66.802" x2="99.03" y2="62.804" width="0" layer="19" extent="1-1"/>
+<wire x1="110.774" y1="122.362" x2="94.966" y2="78.298" width="0" layer="19" extent="1-1"/>
 <wire x1="126.05" y1="137.19" x2="110.774" y2="122.362" width="0" layer="19" extent="1-1"/>
-<wire x1="94.966" y1="78.298" x2="110.774" y2="122.362" width="0" layer="19" extent="1-1"/>
-<wire x1="99.03" y1="62.804" x2="94.966" y2="78.298" width="0" layer="19" extent="1-1"/>
-<wire x1="95.062" y1="62.768" x2="99.03" y2="62.804" width="0" layer="19" extent="1-1"/>
-<wire x1="95.062" y1="57.434" x2="95.062" y2="62.768" width="0" layer="19" extent="1-1"/>
-<wire x1="108.11" y1="45.522" x2="95.062" y2="57.434" width="0" layer="19" extent="1-1"/>
-<wire x1="120.65" y1="66.802" x2="94.966" y2="78.298" width="0" layer="19" extent="1-1"/>
-<wire x1="80.452" y1="38.07" x2="95.062" y2="57.434" width="0" layer="19" extent="1-1"/>
-<wire x1="78.298" y1="22.89" x2="80.452" y2="38.07" width="0" layer="19" extent="1-1"/>
-<wire x1="55.118" y1="8.382" x2="78.298" y2="22.89" width="0" layer="19" extent="1-1"/>
-<wire x1="43.392" y1="5.668" x2="55.118" y2="8.382" width="0" layer="19" extent="1-1"/>
-</signal>
-<signal name="230V">
+</signal>
+<signal name="320V">
 <contactref element="R3" pad="1"/>
-<contactref element="U$11" pad="P$1"/>
-<wire x1="0" y1="-104.14" x2="123.51" y2="126.776" width="0" layer="19" extent="1-1"/>
-</signal>
-<signal name="320V">
+<contactref element="R24" pad="1"/>
+<contactref element="CY2" pad="+"/>
+<wire x1="-63.754" y1="-129.794" x2="123.51" y2="126.776" width="0" layer="19" extent="1-1"/>
+<wire x1="-59.182" y1="-199.898" x2="-63.754" y2="-129.794" width="0" layer="19" extent="1-1"/>
+</signal>
+<signal name="370V">
 <contactref element="R5" pad="1"/>
-<contactref element="U$12" pad="P$1"/>
-<wire x1="0" y1="-106.68" x2="82.108" y2="100.106" width="0" layer="19" extent="1-1"/>
+<contactref element="R24" pad="2"/>
+<contactref element="R23" pad="1"/>
+<contactref element="CY1" pad="+"/>
+<wire x1="-53.594" y1="-129.794" x2="-63.754" y2="-124.46" width="0" layer="19" extent="1-1"/>
+<wire x1="-59.182" y1="-217.932" x2="-53.594" y2="-129.794" width="0" layer="19" extent="1-1"/>
+<wire x1="82.108" y1="100.106" x2="-53.594" y2="-129.794" width="0" layer="19" extent="1-1"/>
 </signal>
 <signal name="477V">
 <contactref element="R10" pad="1"/>
 <contactref element="R9" pad="2"/>
-<contactref element="U$13" pad="P$1"/>
-<contactref element="U$16" pad="P$1"/>
-<wire x1="36.336" y1="59.262" x2="72.818" y2="90.184" width="0" layer="19" extent="1-1"/>
-<wire x1="0" y1="-109.22" x2="36.336" y2="59.262" width="0" layer="19" extent="1-1"/>
-<wire x1="0" y1="-116" x2="0" y2="-109.22" width="0" layer="19" extent="1-1"/>
+<contactref element="R23" pad="2"/>
+<contactref element="R25" pad="1"/>
+<contactref element="CY4" pad="+"/>
+<wire x1="-59.182" y1="-235.966" x2="-63.754" y2="-189.23" width="0" layer="19" extent="1-1"/>
+<wire x1="-53.594" y1="-124.46" x2="-63.754" y2="-189.23" width="0" layer="19" extent="1-1"/>
+<wire x1="36.336" y1="59.262" x2="-53.594" y2="-124.46" width="0" layer="19" extent="1-1"/>
+<wire x1="72.818" y1="90.184" x2="36.336" y2="59.262" width="0" layer="19" extent="1-1"/>
 </signal>
 <signal name="N$8" class="1">
@@
 <contactref element="U$9" pad="P$1"/>
 </signal>
-<signal name="505V">
+<signal name="530V">
 <contactref element="U$18" pad="P$1"/>
+<contactref element="R25" pad="2"/>
+<wire x1="-0.508" y1="-119.634" x2="-53.594" y2="-189.23" width="0" layer="19" extent="1-1"/>
 </signal>
 </signals>
