File: Projects/RingerPro/RingerPro.brd (EAGLE design)
At the start: 31 x 30.4 mm, 43 parts, among them IC1 LIS2DW12TR, P33 TESTPOINT_22, U2 REG710, U3 BSS138BKW, U4 MCP73831T-2ACI_OT, U5 LPS22HDTR, U6 LPS22HDTR, U7 LPS22HDTR

Commit message: Added stuff on RingerPro
Parts:
- added D1: BLUE, SparkFun-LED:LED-0603
- added R8: 100, Passives:R0603
- added R9: 500, Passives:R0603
- added SPST1: PTS526SK08, SPST:PTS526SKG15SMTR2LFS
- C6: device Passives:C0805 -> Passives:C0603
- R3: device Passives:R0805 -> Passives:R0603
- U5, U6, U7: value LPS22HDTR -> LPS22HBTR
- moved C11 2.47 mm to (27.4, 27.8), turned to 270 degrees
- moved P33 1.20 mm to (11.4, 7.75)
- moved U3 1.14 mm to (29.1, 11.2)
- moved R3 1.14 mm to (29.5, 4.95)
- moved R2 1.09 mm to (26.3, 10.9)
- moved U5 1.09 mm to (25.0, 27.8), turned to 270 degrees
- moved C6 1.02 mm to (26.9, 4.95)
Connections:
- new net BTN1: SPST1.3, SPST1.4, U1.P40
- new net LED_B: R9.2, U1.P41
- new net N$11: D1.A, R9.1
- new net N$8: R8.1, U3.3
- net GND: now also D1.C, SPST1.1, SPST1.2
- net VIN: now also R8.2; no longer U3.3
Routing:
- net BTN1: track 0.00 -> 23.5 mm, vias 0 -> 3
- net LED_B: track 0.00 -> 6.96 mm, vias 0 -> 1
- net SCL2: track 40.4 -> 44.2 mm
- net VDD: track 101.6 -> 98.4 mm, vias 7 -> 5
- net VIN: track 44.6 -> 41.8 mm
- net N$8: track 0.00 -> 2.56 mm
- net N$11: track 0.00 -> 2.55 mm
- net !PWM1: track 16.3 -> 17.4 mm
- net N$2: track 3.21 -> 2.07 mm
- net N$1: track 3.09 -> 2.07 mm
- net INT_U7: track 26.4 -> 27.3 mm
- net SDA2: track 40.4 -> 41.0 mm
- net INT_U5: track 38.6 -> 38.0 mm
