File: Projects/RingerPro/RingerPro.sch (EAGLE design)
At the start: 43 parts, among them IC1 LIS2DW12TR, P33 TESTPOINT_22, U2 REG710, U3 BSS138BKW, U4 MCP73831T-2ACI_OT, U5 LPS22HDTR, U6 LPS22HDTR, U7 LPS22HDTR

Commit message: Added stuff on RingerPro
Parts:
- added D1: BLUE, SparkFun-LED:LED-BLUE0603
- added R8: 100, Passives:RESISTOR0603
- added R9: 500, Passives:RESISTOR0603
- added SPST1: PTS526SK08, SPST:PTS526SK08
- C6: device Passives:CAPACITOR0805 -> Passives:CAPACITOR0603
- R3: device Passives:RESISTOR0805 -> Passives:RESISTOR0603
- U5, U6, U7: value LPS22HDTR -> LPS22HBTR
Connections:
- new net BTN1: SPST1.P$2, U1.P0.22
- new net LED_B: R9.2, U1.P0.23
- new net N$11: D1.A, R9.1
- new net N$8: R8.1, U3.D
- net GND: now also D1.C, SPST1.P$1
- net VIN: now also R8.2; no longer U3.D
Changed lines of the file:
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@@
 <layer number="230" name="230bmp" color="7" fill="1" visible="yes" active="yes"/>
 <layer number="231" name="231bmp" color="7" fill="1" visible="yes" active="yes"/>
+<layer number="232" name="Eagle3D_PG2" color="7" fill="1" visible="no" active="no"/>
+<layer number="233" name="Eagle3D_PG3" color="7" fill="1" visible="no" active="no"/>
 <layer number="248" name="Housing" color="7" fill="1" visible="yes" active="yes"/>
 <layer number="249" name="Edge" color="7" fill="1" visible="yes" active="yes"/>
@@
 <part name="U$21" library="PowerSupplies" deviceset="GND" device=""/>
 <part name="U$22" library="PowerSupplies" deviceset="VIN" device=""/>
-<part name="U$23" library="USB" deviceset="ZX80B5P" device=""/>
+<part name="U$23" library="USB" deviceset="ZX80B5P" device="" override_package3d_urn="urn:adsk.eagle:package:23814005/2" override_package_urn="urn:adsk.eagle:footprint:23814006/1"/>
 <part name="U$24" library="PowerSupplies" deviceset="GND" device=""/>
 <part name="C10" library="Passives" deviceset="CAPACITOR" device="0603" value="10uF"/>
 <part name="U3" library="BSS138" deviceset="BSS138BKW" device=""/>
 <part name="U$9" library="PowerSupplies" deviceset="GND" device=""/>
-<part name="C6" library="Passives" deviceset="CAPACITOR" device="0805" value="10uF"/>
-<part name="R3" library="Passives" deviceset="RESISTOR" device="0805" value="100"/>
+<part name="C6" library="Passives" deviceset="CAPACITOR" device="0603" value="10uF"/>
+<part name="R3" library="Passives" deviceset="RESISTOR" device="0603" value="100"/>
 <part name="IC1" library="Accelerometers" deviceset="LIS2DW12TR" device=""/>
 <part name="U$26" library="PowerSupplies" deviceset="GND" device=""/>
@@
 <part name="VDD" library="test_points" deviceset="TESTPOINT_22" device=""/>
 <part name="P33" library="test_points" deviceset="TESTPOINT_22" device=""/>
-<part name="U5" library="Pressure" deviceset="LPS22HDTR" device=""/>
-<part name="U6" library="Pressure" deviceset="LPS22HDTR" device=""/>
+<part name="U5" library="Pressure" deviceset="LPS22HDTR" device="" override_package3d_urn="urn:adsk.eagle:package:23814083/2" override_package_urn="urn:adsk.eagle:footprint:23814084/1" value="LPS22HBTR"/>
+<part name="U6" library="Pressure" deviceset="LPS22HDTR" device="" override_package3d_urn="urn:adsk.eagle:package:23814078/2" override_package_urn="urn:adsk.eagle:footprint:23814079/1" value="LPS22HBTR"/>
 <part name="U$11" library="PowerSupplies" deviceset="VDD" device=""/>
 <part name="U$25" library="PowerSupplies" deviceset="GND" device=""/>
-<part name="U7" library="Pressure" deviceset="LPS22HDTR" device=""/>
+<part name="U7" library="Pressure" deviceset="LPS22HDTR" device="" override_package3d_urn="urn:adsk.eagle:package:23814087/2" override_package_urn="urn:adsk.eagle:footprint:23814088/1" value="LPS22HBTR"/>
 <part name="U$29" library="PowerSupplies" deviceset="VDD" device=""/>
 <part name="C5" library="Passives" deviceset="CAPACITOR" device="0603" value="100nF"/>
@@
 <part name="R6" library="Passives" deviceset="RESISTOR" device="0603" value="10k"/>
 <part name="R7" library="Passives" deviceset="RESISTOR" device="0603" value="10k"/>
+<part name="R8" library="Passives" deviceset="RESISTOR" device="0603" value="100"/>
+<part name="SPST1" library="SPST" deviceset="PTS526SK08" device="" override_package3d_urn="urn:adsk.eagle:package:23850826/2" override_package_urn="urn:adsk.eagle:footprint:23850877/1"/>
+<part name="D1" library="SparkFun-LED" deviceset="LED-BLUE" device="0603" value="BLUE"/>
+<part name="U$30" library="PowerSupplies" deviceset="GND" device=""/>
+<part name="U$31" library="PowerSupplies" deviceset="GND" device=""/>
+<part name="R9" library="Passives" deviceset="RESISTOR" device="0603" value="500"/>
 </parts>
 <sheets>
@@
 </instance>
 <instance part="U$5" gate="GND" x="-116.84" y="-68.58" smashed="yes" grouprefs="DCDC"/>
-<instance part="U$4" gate="G$1" x="-30.48" y="101.6" smashed="yes" grouprefs="CLASS_D"/>
+<instance part="U$4" gate="G$1" x="-30.48" y="106.68" smashed="yes" grouprefs="CLASS_D"/>
 <instance part="C2" gate="G$1" x="-152.4" y="-30.48" smashed="yes" rot="R90" grouprefs="DCDC">
 <attribute name="NAME" x="-152.781" y="-28.956" size="1.778" layer="95" rot="R90"/>
@@
 <attribute name="NAME" x="46.736" y="-46.7614" size="0.6096" layer="95"/>
 <attribute name="VALUE" x="46.736" y="-50.292" size="0.6096" layer="96"/>
+</instance>
+<instance part="R8" gate="G$1" x="-30.48" y="93.98" smashed="yes" rot="R90">
+<attribute name="NAME" x="-31.9786" y="92.456" size="0.6096" layer="95" rot="R90"/>
+<attribute name="VALUE" x="-28.448" y="92.456" size="0.6096" layer="96" rot="R90"/>
+</instance>
+<instance part="SPST1" gate="G$1" x="116.84" y="-35.56" smashed="yes" rot="R90"/>
+<instance part="D1" gate="G$1" x="132.08" y="-38.1" smashed="yes">
+<attribute name="NAME" x="128.651" y="-42.672" size="1.778" layer="95" font="vector" rot="R90"/>
+<attribute name="VALUE" x="133.985" y="-42.672" size="1.778" layer="96" font="vector" rot="R90" align="top-left"/>
+</instance>
+<instance part="U$30" gate="GND" x="116.84" y="-53.34" smashed="yes"/>
+<instance part="U$31" gate="GND" x="132.08" y="-53.34" smashed="yes"/>
+<instance part="R9" gate="G$1" x="132.08" y="-25.4" smashed="yes" rot="R90">
+<attribute name="NAME" x="130.5814" y="-26.924" size="0.6096" layer="95" rot="R90"/>
+<attribute name="VALUE" x="134.112" y="-26.924" size="0.6096" layer="96" rot="R90"/>
 </instance>
 </instances>
@@
 <wire x1="-157.48" y1="68.58" x2="-152.4" y2="68.58" width="0.1524" layer="91" grouprefs="CHARGER"/>
 <junction x="-152.4" y="68.58"/>
-</segment>
-<segment>
-<pinref part="U3" gate="G$1" pin="S"/>
-<pinref part="U$9" gate="GND" pin="GND"/>
-<wire x1="-30.48" y1="76.2" x2="-30.48" y2="71.12" width="0.1524" layer="91" grouprefs="CLASS_D"/>
 </segment>
 <segment>
@@
 <wire x1="106.68" y1="30.48" x2="101.6" y2="30.48" width="0.1524" layer="91" grouprefs="PRESSURE"/>
 </segment>
+<segment>
+<pinref part="U$9" gate="GND" pin="GND"/>
+<pinref part="U3" gate="G$1" pin="S"/>
+<wire x1="-30.48" y1="71.12" x2="-30.48" y2="76.2" width="0.1524" layer="91"/>
+</segment>
+<segment>
+<pinref part="U$30" gate="GND" pin="GND"/>
+<pinref part="SPST1" gate="G$1" pin="P$1"/>
+<wire x1="116.84" y1="-50.8" x2="116.84" y2="-43.18" width="0.1524" layer="91"/>
+</segment>
+<segment>
+<pinref part="D1" gate="G$1" pin="C"/>
+<pinref part="U$31" gate="GND" pin="GND"/>
+<wire x1="132.08" y1="-43.18" x2="132.08" y2="-50.8" width="0.1524" layer="91"/>
+</segment>
 </net>
 <net name="VIN" class="0">
@@
 </segment>
 <segment>
+<pinref part="R8" gate="G$1" pin="2"/>
 <pinref part="U$4" gate="G$1" pin="VIN"/>
-<wire x1="-30.48" y1="86.36" x2="-30.48" y2="91.44" width="0.1524" layer="91" grouprefs="CLASS_D"/>
-<pinref part="U3" gate="G$1" pin="D"/>
+<wire x1="-30.48" y1="99.06" x2="-30.48" y2="101.6" width="0.1524" layer="91"/>
 <pinref part="R3" gate="G$1" pin="2"/>
-<wire x1="-30.48" y1="91.44" x2="-30.48" y2="99.06" width="0.1524" layer="91" grouprefs="CLASS_D"/>
-<wire x1="-17.78" y1="91.44" x2="-30.48" y2="91.44" width="0.1524" layer="91"/>
-<junction x="-30.48" y="91.44"/>
+<wire x1="-30.48" y1="101.6" x2="-30.48" y2="104.14" width="0.1524" layer="91"/>
+<wire x1="-17.78" y1="91.44" x2="-22.86" y2="91.44" width="0.1524" layer="91"/>
+<wire x1="-22.86" y1="91.44" x2="-22.86" y2="101.6" width="0.1524" layer="91"/>
+<wire x1="-22.86" y1="101.6" x2="-30.48" y2="101.6" width="0.1524" layer="91"/>
+<junction x="-30.48" y="101.6"/>
 </segment>
 </net>
@@
 </segment>
 </net>
+<net name="N$8" class="0">
+<segment>
+<pinref part="U3" gate="G$1" pin="D"/>
+<pinref part="R8" gate="G$1" pin="1"/>
+<wire x1="-30.48" y1="86.36" x2="-30.48" y2="88.9" width="0.1524" layer="91"/>
+</segment>
+</net>
+<net name="N$11" class="0">
+<segment>
+<pinref part="D1" gate="G$1" pin="A"/>
+<pinref part="R9" gate="G$1" pin="1"/>
+<wire x1="132.08" y1="-35.56" x2="132.08" y2="-30.48" width="0.1524" layer="91"/>
+</segment>
+</net>
+<net name="BTN1" class="0">
+<segment>
+<pinref part="SPST1" gate="G$1" pin="P$2"/>
+<wire x1="116.84" y1="-35.56" x2="116.84" y2="-15.24" width="0.1524" layer="91"/>
+<label x="116.84" y="-15.24" size="1.27" layer="95" rot="R90" xref="yes"/>
+</segment>
+<segment>
+<pinref part="U1" gate="G$1" pin="P0.22"/>
+<wire x1="12.7" y1="-5.08" x2="22.86" y2="-5.08" width="0.1524" layer="91"/>
+<label x="22.86" y="-5.08" size="1.27" layer="95" xref="yes"/>
+</segment>
+</net>
+<net name="LED_B" class="0">
+<segment>
+<pinref part="R9" gate="G$1" pin="2"/>
+<wire x1="132.08" y1="-20.32" x2="132.08" y2="-15.24" width="0.1524" layer="91"/>
+<label x="132.08" y="-15.24" size="1.27" layer="95" rot="R90" xref="yes"/>
+</segment>
+<segment>
+<pinref part="U1" gate="G$1" pin="P0.23"/>
+<wire x1="12.7" y1="-2.54" x2="22.86" y2="-2.54" width="0.1524" layer="91"/>
+<label x="22.86" y="-2.54" size="1.27" layer="95" xref="yes"/>
+</segment>
+</net>
 </nets>
 </sheet>
@@
 </drawing>
 <compatibility>
+<note version="8.3" severity="warning">
+Since Version 8.3, EAGLE supports the association of 3D packages
+with devices in libraries, schematics, and board files. Those 3D
+packages will not be understood (or retained) with this version.
+</note>
 <note version="9.5" severity="warning">
 Since Version 9.5, EAGLE supports persistent groups with
@@
 will not be understood (or retained) with this version.
 </note>
+<note version="9.4" severity="warning">
+Since Version 9.4, EAGLE supports the overriding of 3D packages
+in schematics and board files. Those overridden 3d packages
+will not be understood (or retained) with this version.
+</note>
